Commit message: box_confirm

File: Gazebo_ws/src/gazebo_sim/urdf/box.urdf (robot description, URDF)
Before this commit: robot box_robot, 1 links, 0 joints
Links:
- link base_link: mass 1.0 -> 1000; geometry collision box size=1 1 1; visual box size=1 1 1

Commit message: Finally_Moves

File: Gazebo_ws/src/gazebo_sim/urdf/box.urdf (robot description, URDF)
Before this commit: robot box_robot, 1 links, 0 joints
Links:
- added link robot_base, mass 1000; collision box size=1 1 1; visual box size=1 1 1
- link base_link: mass 1000 -> None; geometry 
Joints:
- added joint base_joint: type fixed, parent base_link, child robot_base, origin xyz=0 0 0 rpy=0 0 0

Commit message: 放弃，提交。

File: Gazebo_ws/src/gazebo_sim/urdf/box.urdf (robot description, URDF)
Before this commit: robot box_robot, 2 links, 1 joints
Links:
- removed link robot_base
- link base_link: mass None -> 1000; geometry collision box size=1 1 1; visual box size=1 1 1
Joints:
- removed joint base_joint
